File: ovc5/hardware/carrier/interfaces.kicad_sch (KiCad schematic)
At the start: 34 parts, among them J3 Micro_SD_Card_Det_Hirose_DM3AT, J5 Conn_01x04, J6 Conn_02x06_Odd_Even, J7 Conn_01x04, J8 Conn_01x04, J9 Conn_01x04, SW1 SW_DIP_x03, U11 ARJ11C-MBSAS-A-BA-7MU2, U12 FT232RL, U13 TXS02612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

Commit message: Start working on FIXME for revb
Signed-off-by: Luca Della Vedova <luca@openrobotics.org>
Parts:
- SW1: D1PN CT2193MST-ND -> 563-CFS-0300TACT-ND; MFN CTS -> Nidec Copal Electronics; MPN 219-3MST -> CFS-0300TA
Changed lines of the file:
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@@
       (effects (font (size 1.27 1.27)) hide)
     )
-    (property "D1PN" "CT2193MST-ND" (id 5) (at 115.57 171.45 0)
+    (property "D1PN" "563-CFS-0300TACT-ND" (id 5) (at 115.57 171.45 0)
       (effects (font (size 1.27 1.27)) hide)
     )
-    (property "MFN" "CTS" (id 6) (at 115.57 171.45 0)
+    (property "MFN" "Nidec Copal Electronics" (id 6) (at 115.57 171.45 0)
       (effects (font (size 1.27 1.27)) hide)
     )
-    (property "MPN" "219-3MST" (id 7) (at 115.57 171.45 0)
+    (property "MPN" "CFS-0300TA" (id 7) (at 115.57 171.45 0)
       (effects (font (size 1.27 1.27)) hide)
     )
