File: ovc5/hardware/carrier/usb.kicad_sch (KiCad schematic)
At the start: 108 parts, among them J1 USB_C_Receptacle, U10 S25FL064, U2 CYUSB43x7, U5 USB3_A_Dual_Stacked, U8 TPS2561, Y1 25MHz

Commit message: Start working on FIXME for revb
Signed-off-by: Luca Della Vedova <luca@openrobotics.org>
Connections:
- net FPGA_USB0_RX+: now also U2.P12 (TX1_P3_P); no longer U2.N13 (RX1_P3_P)
- net FPGA_USB0_RX-: now also U2.P13 (TX1_P3_N); no longer U2.N14 (RX1_P3_N)
- net FPGA_USB0_TX+: now also U2.N13 (RX1_P3_P); no longer U2.P13 (TX1_P3_N)
- net FPGA_USB0_TX-: now also U2.N14 (RX1_P3_N); no longer U2.P12 (TX1_P3_P)
- net FPGA_USB1_RX+: now also U2.H13 (TX_P4_N); no longer U2.G13 (RX_P4_N)
- net FPGA_USB1_RX-: now also U2.H14 (TX_P4_P); no longer U2.G14 (RX_P4_P)
- net FPGA_USB1_TX+: now also U2.G13 (RX_P4_N); no longer U2.H13 (TX_P4_N)
- net FPGA_USB1_TX-: now also U2.G14 (RX_P4_P); no longer U2.H14 (TX_P4_P)
- net USB_DS_D_N: no longer D3.2 (A2), J1.A7 (D-), J1.B7 (D-)
- net USB_DS_D_P: no longer D3.1 (A1), J1.A6 (D+), J1.B6 (D+)
- net USB_DS_RX1_N: no longer J1.B10 (RX1-)
- net USB_DS_RX1_P: no longer J1.B11 (RX1+)
- net USB_DS_RX2_N: no longer J1.A10 (RX2-)
- net USB_DS_RX2_P: no longer J1.A11 (RX2+)
- net USB_DS_TX1_N: no longer C76.2
- net USB_DS_TX1_P: no longer C74.2
- net USB_DS_TX2_N: no longer C77.2
- net USB_DS_TX2_P: no longer C75.2
- net USB_H1_D_N: now also U2.J2 (D_P5_N); no longer U2.J1 (D_P5_P)
- net USB_H1_D_P: now also U2.J1 (D_P5_P); no longer U2.J2 (D_P5_N)
- net USB_DS1_CC1: now reaches U2.L8 (CC1_P3)
- net USB_DS1_CC1: now also R20.1
- net USB_DS_CC1 renamed USB_US_CC1
- net USB_DS_CC2 renamed USB_US_CC2
- net USB_DS_TX1_CONN_N renamed USB_US_TX1_CONN_N
- net USB_DS_TX1_CONN_P renamed USB_US_TX1_CONN_P
- net USB_DS_TX2_CONN_N renamed USB_US_TX2_CONN_N
- net USB_DS_TX2_CONN_P renamed USB_US_TX2_CONN_P
- net USB_US0_CC1 renamed USB_DS0_CC1
- net USB_US1_CC1: no longer names the net of U2.K9 (CC1_P2)
- net USB_US1_CC1: no longer R20.1
- new net USB_US_D_N: D3.2 (A2), J1.A7 (D-), J1.B7 (D-)
- new net USB_US_D_P: D3.1 (A1), J1.A6 (D+), J1.B6 (D+)
- new net USB_US_RX1_N: J1.B10 (RX1-)
- new net USB_US_RX1_P: J1.B11 (RX1+)
- new net USB_US_RX2_N: J1.A10 (RX2-)
- new net USB_US_RX2_P: J1.A11 (RX2+)
- new net USB_US_TX1_N: C76.2
- new net USB_US_TX1_P: C74.2
- new net USB_US_TX2_N: C77.2
- new net USB_US_TX2_P: C75.2
